File: splitter.brd (EAGLE design)
At the start: 23.8 x 17.8 mm, 16 parts

Commit message: cosmetic changes on the board layout
Parts:
- moved R3 0.95 mm to (18.4, 12.1)
- moved C1 0.13 mm to (6.99, 10.6)
Routing:
- net N$7: track 11.7 -> 11.2 mm
Other:
- board size 23.8 x 17.8 mm -> 23.6 x 17.8 mm

Commit message: last minute changes
Routing:
- net VCC: track 54.1 -> 53.1 mm
Changed lines of the file:
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@@
 <setting verticaltext="up"/>
 </settings>
-<grid distance="25" unitdist="mil" unit="mm" style="lines" multiple="1" display="no" altdistance="5" altunitdist="mil" altunit="mil"/>
+<grid distance="25" unitdist="mil" unit="mil" style="lines" multiple="1" display="no" altdistance="12.5" altunitdist="mil" altunit="mil"/>
 <layers>
-<layer number="1" name="Top" color="4" fill="1" visible="no" active="yes"/>
-<layer number="16" name="Bottom" color="1" fill="1" visible="yes" active="yes"/>
+<layer number="1" name="Top" color="4" fill="1" visible="yes" active="yes"/>
+<layer number="16" name="Bottom" color="1" fill="1" visible="no" active="yes"/>
 <layer number="17" name="Pads" color="2" fill="1" visible="yes" active="yes"/>
 <layer number="18" name="Vias" color="2" fill="1" visible="yes" active="yes"/>
 <layer number="19" name="Unrouted" color="6" fill="1" visible="yes" active="yes"/>
 <layer number="20" name="Dimension" color="15" fill="1" visible="yes" active="yes"/>
-<layer number="21" name="tPlace" color="7" fill="1" visible="no" active="yes"/>
-<layer number="22" name="bPlace" color="7" fill="1" visible="yes" active="yes"/>
-<layer number="23" name="tOrigins" color="15" fill="1" visible="no" active="yes"/>
-<layer number="24" name="bOrigins" color="15" fill="1" visible="yes" active="yes"/>
-<layer number="25" name="tNames" color="7" fill="1" visible="no" active="yes"/>
-<layer number="26" name="bNames" color="7" fill="1" visible="yes" active="yes"/>
-<layer number="27" name="tValues" color="7" fill="1" visible="no" active="yes"/>
-<layer number="28" name="bValues" color="7" fill="1" visible="yes" active="yes"/>
+<layer number="21" name="tPlace" color="7" fill="1" visible="yes" active="yes"/>
+<layer number="22" name="bPlace" color="7" fill="1" visible="no" active="yes"/>
+<layer number="23" name="tOrigins" color="15" fill="1" visible="yes" active="yes"/>
+<layer number="24" name="bOrigins" color="15" fill="1" visible="no" active="yes"/>
+<layer number="25" name="tNames" color="7" fill="1" visible="yes" active="yes"/>
+<layer number="26" name="bNames" color="7" fill="1" visible="no" active="yes"/>
+<layer number="27" name="tValues" color="7" fill="1" visible="yes" active="yes"/>
+<layer number="28" name="bValues" color="7" fill="1" visible="no" active="yes"/>
 <layer number="29" name="tStop" color="7" fill="3" visible="no" active="yes"/>
 <layer number="30" name="bStop" color="7" fill="6" visible="no" active="yes"/>
@@
 <contactref element="VREG" pad="1"/>
 <contactref element="VREG" pad="3"/>
-<wire x1="4.1275" y1="0.9525" x2="8.255" y2="0.9525" width="0.8128" layer="1"/>
 <wire x1="8.255" y1="0.9525" x2="22.86" y2="0.9525" width="0.8128" layer="1"/>
 <wire x1="4.1275" y1="9.8425" x2="1.778" y2="11.43" width="0.8128" layer="1"/>
 <contactref element="C4" pad="A"/>
 <wire x1="4.1275" y1="9.8425" x2="4.1275" y2="6.35" width="0.8128" layer="1"/>
-<wire x1="4.1275" y1="6.35" x2="4.1275" y2="0.9525" width="0.8128" layer="1"/>
 <wire x1="5.715" y1="6.48" x2="5.585" y2="6.35" width="0.8128" layer="1"/>
 <wire x1="5.585" y1="6.35" x2="4.1275" y2="6.35" width="0.8128" layer="1"/>
@@
 <wire x1="8.2249" y1="3.8125" x2="8.255" y2="3.7824" width="0.6096" layer="1"/>
 <wire x1="8.255" y1="3.7824" x2="8.255" y2="0.9525" width="0.6096" layer="1"/>
+<wire x1="8.255" y1="0.9525" x2="5.715" y2="0.9525" width="0.8128" layer="1"/>
+<wire x1="5.715" y1="0.9525" x2="4.1275" y2="2.54" width="0.8128" layer="1"/>
+<wire x1="4.1275" y1="2.54" x2="4.1275" y2="6.35" width="0.8128" layer="1"/>
 </signal>
 <signal name="N$1">

Commit message: fixed cap values
Parts:
- C3: value 100uf -> 100uF
- C4, C6: value 22uf -> 22uF
Changed lines of the file:
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@@
 <text x="18.415" y="14.2875" size="1.27" layer="26" rot="SMR180">1</text>
 <text x="18.0975" y="6.0325" size="1.27" layer="26" rot="SMR180">2</text>
-<wire x1="22.225" y1="9.525" x2="19.3675" y2="9.525" width="0.6096" layer="24"/>
+<wire x1="22.225" y1="9.525" x2="19.3675" y2="9.525" width="0.6096" layer="26"/>
 <text x="3.81" y="0.635" size="0.8128" layer="25">CC BY-SA 4.0</text>
 <text x="6.35" y="13.97" size="0.8128" layer="26" rot="SMR180">CC BY-SA 4.0</text>
@@
 <attribute name="VALUE" x="16.4195" y="17.4005" size="0.6096" layer="27" rot="R180"/>
 </element>
-<element name="C3" library="SparkFun-Passives" package="EIA3528" value="100uf" x="14.605" y="11.7475" smashed="yes" rot="R180">
+<element name="C3" library="SparkFun-Passives" package="EIA3528" value="100uF" x="14.605" y="11.7475" smashed="yes" rot="R180">
 <attribute name="NAME" x="13.3985" y="9.0645" size="0.8128" layer="25"/>
 <attribute name="VALUE" x="15.4575" y="9.1425" size="0.6096" layer="27"/>
 </element>
-<element name="C6" library="SparkFun-Passives" package="EIA3216" value="22uf" x="10.16" y="8.5725" smashed="yes" rot="R180">
+<element name="C6" library="SparkFun-Passives" package="EIA3216" value="22uF" x="10.16" y="8.5725" smashed="yes" rot="R180">
 <attribute name="NAME" x="6.985" y="9.541" size="0.8128" layer="25" rot="R180"/>
 <attribute name="VALUE" x="7.212" y="8.5105" size="0.6096" layer="27" rot="R180"/>
@@
 <element name="U$2" library="SparkFun-Aesthetics" package="OSHW-LOGO-S" value="" x="1.905" y="1.5875"/>
 <element name="U$3" library="SparkFun-Aesthetics" package="OSHW-LOGO-S" value="" x="9.525" y="10.4775" rot="SMR180"/>
-<element name="C4" library="SparkFun-Passives" package="EIA3216" value="22uf" x="5.715" y="5.08" smashed="yes" rot="R90">
+<element name="C4" library="SparkFun-Passives" package="EIA3216" value="22uF" x="5.715" y="5.08" smashed="yes" rot="R90">
 <attribute name="NAME" x="4.064" y="6.62" size="0.8128" layer="25" rot="R180"/>
 <attribute name="VALUE" x="4.037" y="5.018" size="0.6096" layer="27" rot="R180"/>
